File: BLEkeyboard/BLEKeyboardKicad/BLEkeyboard.kicad_pcb (KiCad board)
At the start: 2 copper layers, 90 x 130 mm, 51 parts, among them J1 Conn_01x02_Socket, SW1 SW_SPDT, SW10 SW_Push, SW11 SW_Push, SW12 SW_Push, SW13 SW_Push, SW14 SW_Push, SW15 SW_Push, SW16 SW_Push, SW17 SW_Push, SW18 SW_Push, SW19 SW_Push, SW2 RotaryEncoder_Switch, SW20 SW_Push, SW3 SW_Push, SW4 SW_Push, SW5 SW_Push, SW6 SW_Push, SW7 SW_Push, SW8 SW_Push, SW9 SW_Push, U1 ER_OLEDM0.91_1x-I2C, U2 XIAO-nRF52840-Plus-SMD

Commit message: fixed mounting hole issues
Parts:
- SW19, SW20: footprint PCM_Switch_Keyboard_Cherry_MX:SW_Cherry_MX_PCB_2.00u -> BLEKeyboardKicad:CherryMX_2.00u_PCB_StabWireBottom
- moved H4 3.80 mm to (169.8, 145.8)
- moved H3 0.75 mm to (89.0, 145.8)
- moved D12 0.54 mm to (145.5, 81.5)
- moved D13 0.41 mm to (145.5, 100.6)
- moved D14 0.41 mm to (145.5, 119.8)
- moved D15 0.41 mm to (145.5, 139.0)
- moved H1 0.19 mm to (89.0, 24.2)
Routing:
- net /3v3: track 27.2 -> 34.9 mm, vias 0 -> 2
- net GND: track 39.4 -> 36.0 mm
- net /row2: track 114.5 -> 115.9 mm
- net /row1: track 95.7 -> 97.1 mm
- net /row0: track 76.8 -> 78.0 mm
- net /XIAO_VBAT: track 76.5 -> 75.3 mm, vias 2 -> 0
- net /col1: track 116.5 -> 117.3 mm
- net /col2: track 99.0 -> 99.8 mm
- net Net-(D12-A): track 13.6 -> 13.0 mm
