File: BLEkeyboard/BLEKeyboardKicad/BLEkeyboard.kicad_sch (KiCad schematic)
At the start: 49 parts, among them J1 Conn_01x02_Socket, SW1 SW_SPDT, SW10 SW_Push, SW11 SW_Push, SW12 SW_Push, SW13 SW_Push, SW14 SW_Push, SW15 SW_Push, SW16 SW_Push, SW17 SW_Push, SW18 SW_Push, SW19 SW_Push, SW2 RotaryEncoder_Switch, SW20 SW_Push, SW3 SW_Push, SW4 SW_Push, SW5 SW_Push, SW6 SW_Push, SW7 SW_Push, SW8 SW_Push, SW9 SW_Push, U1 ER_OLEDM0.91_1x-I2C, U2 XIAO-nRF52840-Plus-SMD

Commit message: fixed mounting hole issues
Parts:
- SW19, SW20: footprint PCM_Switch_Keyboard_Cherry_MX:SW_Cherry_MX_PCB_2.00u -> BLEKeyboardKicad:CherryMX_2.00u_PCB_StabWireBottom
Other:
- note added: "XIAO-NRF52840PLUS + ON/OFF Switch"
- note removed: "MCU"
Changed lines of the file:
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@@
 		)
 	)
-	(text "MCU"
+	(text "XIAO-NRF52840PLUS + ON/OFF Switch"
 		(exclude_from_sim no)
-		(at 93.726 26.416 0)
+		(at 109.728 22.352 0)
 		(effects
 			(font
@@
 		(dnp no)
 		(fields_autoplaced yes)
-		(property "Reference" "#PWR06"
+		(property "Reference" "#PWR07"
 			(at 158.75 106.68 0)
 			(hide yes)
@@
 			(project "BLEkeyboard"
 				(path "/a8b51667-118e-4d88-a968-30985fdb56f2"
-					(reference "#PWR06")
+					(reference "#PWR07")
 					(unit 1)
 				)
@@
 			)
 		)
-		(property "Footprint" "PCM_Switch_Keyboard_Cherry_MX:SW_Cherry_MX_PCB_2.00u"
+		(property "Footprint" "BLEKeyboardKicad:CherryMX_2.00u_PCB_StabWireBottom"
 			(at 267.97 87.63 0)
 			(hide yes)
@@
 		(in_pos_files yes)
 		(dnp no)
-		(property "Reference" "#PWR09"
+		(property "Reference" "#PWR04"
 			(at 111.76 123.19 0)
 			(hide yes)
@@
 			(project "BLEkeyboard"
 				(path "/a8b51667-118e-4d88-a968-30985fdb56f2"
-					(reference "#PWR09")
+					(reference "#PWR04")
 					(unit 1)
 				)
@@
 			)
 		)
-		(property "Footprint" "PCM_Switch_Keyboard_Cherry_MX:SW_Cherry_MX_PCB_2.00u"
+		(property "Footprint" "BLEKeyboardKicad:CherryMX_2.00u_PCB_StabWireBottom"
 			(at 267.97 49.53 0)
 			(hide yes)
@@
 		(dnp no)
 		(fields_autoplaced yes)
-		(property "Reference" "#PWR07"
+		(property "Reference" "#PWR08"
 			(at 165.1 44.45 0)
 			(hide yes)
@@
 			(project "BLEkeyboard"
 				(path "/a8b51667-118e-4d88-a968-30985fdb56f2"
-					(reference "#PWR07")
+					(reference "#PWR08")
 					(unit 1)
 				)
@@
 		(dnp no)
 		(fields_autoplaced yes)
-		(property "Reference" "#PWR08"
+		(property "Reference" "#PWR09"
 			(at 185.42 57.15 0)
 			(hide yes)
@@
 			(project "BLEkeyboard"
 				(path "/a8b51667-118e-4d88-a968-30985fdb56f2"
-					(reference "#PWR08")
+					(reference "#PWR09")
 					(unit 1)
 				)
@@
 		(in_pos_files yes)
 		(dnp no)
-		(property "Reference" "#PWR04"
+		(property "Reference" "#PWR05"
 			(at 115.57 111.76 0)
 			(hide yes)
@@
 			(project "BLEkeyboard"
 				(path "/a8b51667-118e-4d88-a968-30985fdb56f2"
-					(reference "#PWR04")
+					(reference "#PWR05")
 					(unit 1)
 				)
@@
 		(dnp no)
 		(fields_autoplaced yes)
-		(property "Reference" "#PWR05"
+		(property "Reference" "#PWR06"
 			(at 124.46 142.24 0)
 			(hide yes)
@@
 			(project "BLEkeyboard"
 				(path "/a8b51667-118e-4d88-a968-30985fdb56f2"
-					(reference "#PWR05")
+					(reference "#PWR06")
 					(unit 1)
 				)
